Commit message: FIx de urdf y visualizacion en gazebo

File: install/puzzlebot_description/share/puzzlebot_description/urdf/puzzlebot.urdf (robot description, URDF)
Before this commit: robot Puzzlebot_Jetson_Lidar_Ed, 6 links, 5 joints
Links:
- link base_link: geometry collision mesh filename=package://puzzlebot_description/meshes/Puzzlebot_Jetson_Lid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 scale=1 1 1; visual mesh filename=package://puzzlebot_description/meshes/Puzzlebot_Jetson_Lid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 scale=1 1 1
- link caster_link: geometry collision mesh filename=package://puzzlebot_description/meshes/Puzzlebot_Caster_Whe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 scale=1 1 1; visual mesh filename=package://puzzlebot_description/meshes/Puzzlebot_Caster_Whe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 scale=1 1 1
- link laser_link: geometry collision cylinder length=0.04 radius=0.03; visual cylinder length=0.04 radius=0.03
- link wheel_l_link: geometry collision mesh filename=package://puzzlebot_description/meshes/Puzzlebot_Wheel.stl scale=1 1 1; visual mesh filename=package://puzzlebot_description/meshes/Puzzlebot_Wheel.stl scale=1 1 1
- link wheel_r_link: geometry collision mesh filename=package://puzzlebot_description/meshes/Puzzlebot_Wheel.stl scale=1 1 1; visual mesh filename=package://puzzlebot_description/meshes/Puzzlebot_Wheel.stl scale=1 1 1
