Commit message: Functional_sim

File: puzzlebot_description/urdf/sensor_properties.xacro (robot description, xacro)
@@ -5,5 +5,5 @@
     <!--Puzzlebot parameters-->
         <!--General parameters-->
-            <xacro:property name="wheel_base_distance" value="0.19"/>
+            <xacro:property name="wheel_base_distance" value="0.17"/>
     <!--Chassis-->
         <!--Chassis Inertial/Collision parameters-->
@@ -104,5 +104,5 @@
             <xacro:property name="wheel_mass" value="0.027"/>
             <xacro:property name="wheel_height" value="0.012"/>
-            <xacro:property name="wheel_radius" value="0.05"/>
+            <xacro:property name="wheel_radius" value="0.045"/>
             <xacro:property name="wheel_inertia_pos_x" value="0.0"/>
             <xacro:property name="wheel_inertia_pos_y" value="0.0"/>
