Commit message: description_patch

File: puzzlebot_description/urdf/puzzlebot.urdf.xacro (robot description, xacro)
@@ -1,4 +1,9 @@
 <?xml version="1.0"?>
-<robot name="Puzzlebot_Jetson_Lidar_Ed">
+<robot name="Puzzlebot_Jetson_Lidar_Ed" xmlns:xacro="http://www.ros.org/wiki/xacro">
+  <xacro:include filename="$(find puzzlebot_description)/urdf/sensor.xacro"/>
+  <xacro:include filename="$(find puzzlebot_description)/urdf/macros.xacro"/>
+  <xacro:include filename="$(find puzzlebot_description)/urdf/puzzlebot_control.xacro"/>
+  <xacro:include filename="$(find puzzlebot_description)/urdf/sensor_properties.xacro"/>
+  <xacro:arg name="prefix" default=""/>
   <material name="green"><color rgba="0.0 1.0 0.0 1.0"/></material>
   <material name="black"><color rgba="0.0 0.0 0.0 1.0"/></material>
@@ -12,5 +17,5 @@
       <origin xyz="0 0 0" rpy="0 0 0"/>
       <geometry>
-        <mesh filename="package://puzzlebot_description/meshes/Puzzlebot_Jetson_Lidar_Edition_Base.stl" scale="1 1 1"/>
+        <mesh filename="file://$(find puzzlebot_description)/meshes/Puzzlebot_Jetson_Lidar_Edition_Base.stl" scale="1 1 1"/>
       </geometry>
       <material name="green"/>
@@ -19,5 +24,5 @@
       <origin xyz="0 0 0" rpy="0 0 0"/>
       <geometry>
-        <mesh filename="package://puzzlebot_description/meshes/Puzzlebot_Jetson_Lidar_Edition_Base.stl" scale="1 1 1"/>
+        <mesh filename="file://$(find puzzlebot_description)/meshes/Puzzlebot_Jetson_Lidar_Edition_Base.stl" scale="1 1 1"/>
       </geometry>
     </collision>
@@ -31,5 +36,5 @@
       <origin xyz="0 0 0" rpy="-1.5708 0 0"/>
       <geometry>
-        <mesh filename="package://puzzlebot_description/meshes/Puzzlebot_Wheel.stl" scale="1 1 1"/>
+        <mesh filename="file://$(find puzzlebot_description)/meshes/Puzzlebot_Wheel.stl" scale="1 1 1"/>
       </geometry>
       <material name="green"/>
@@ -38,5 +43,5 @@
       <origin xyz="0 0 0" rpy="-1.5708 0 0"/>
       <geometry>
-        <mesh filename="package://puzzlebot_description/meshes/Puzzlebot_Wheel.stl" scale="1 1 1"/>
+        <mesh filename="file://$(find puzzlebot_description)/meshes/Puzzlebot_Wheel.stl" scale="1 1 1"/>
       </geometry>
     </collision>
@@ -50,5 +55,5 @@
       <origin xyz="0 0 0" rpy="1.5708 0 0"/>
       <geometry>
-        <mesh filename="package://puzzlebot_description/meshes/Puzzlebot_Wheel.stl" scale="1 1 1"/>
+        <mesh filename="file://$(find puzzlebot_description)/meshes/Puzzlebot_Wheel.stl" scale="1 1 1"/>
       </geometry>
       <material name="green"/>
@@ -57,5 +62,5 @@
       <origin xyz="0 0 0" rpy="1.5708 0 0"/>
       <geometry>
-        <mesh filename="package://puzzlebot_description/meshes/Puzzlebot_Wheel.stl" scale="1 1 1"/>
+        <mesh filename="file://$(find puzzlebot_description)/meshes/Puzzlebot_Wheel.stl" scale="1 1 1"/>
       </geometry>
     </collision>
@@ -68,5 +73,5 @@
     <visual>
       <geometry>
-        <mesh filename="package://puzzlebot_description/meshes/Puzzlebot_Caster_Wheel.stl" scale="1 1 1"/>
+        <mesh filename="file://$(find puzzlebot_description)/meshes/Puzzlebot_Caster_Wheel.stl" scale="1 1 1"/>
       </geometry>
       <material name="green"/>
@@ -74,5 +79,5 @@
     <collision>
       <geometry>
-        <mesh filename="package://puzzlebot_description/meshes/Puzzlebot_Caster_Wheel.stl" scale="1 1 1"/>
+        <mesh filename="file://$(find puzzlebot_description)/meshes/Puzzlebot_Caster_Wheel.stl" scale="1 1 1"/>
       </geometry>
     </collision>
@@ -186,3 +191,6 @@
     <material>Gazebo/Green</material>
   </gazebo>
+  <xacro:include filename="$(find puzzlebot_description)/urdf/sensor.xacro"/>
+  <xacro:puzzlebot_control prefix="$(arg prefix)"/>
+  <xacro:rpi_lidar_sensor prefix="$(arg prefix)"/>
 </robot>

File: puzzlebot_description/urdf/puzzlebot_control.xacro (robot description, xacro)
@@ -1,28 +1,31 @@
-<?xml version ="1.0?>
+<?xml version="1.0"?>
 <robot xmlns:xacro="http://www.ros.org/wiki/xacro">
     <xacro:macro name="puzzlebot_control" params="prefix">
         <gazebo>
-            <plugin filename="gz-sim-sensors-system" name="gz::sim::systems::Sensors"/>
+            <plugin filename="gz-sim-sensors-system"
+                    name="ignition::gazebo::systems::Sensors">
                 <render_engine>ogre2</render_engine>
             </plugin>
-            <plugin filename="gz-sim-diff-drive-systems" name="gz::sim::systems::DiffDrive"/>
-                <left_joint>${prefix}wheel_left_joint</left_joint>          # the joints that will be controlled by the plugin
-                <right_joint>${prefix}wheel_right_joint</right_joint>       # the joints that will be controlled by the plugin
-                <wheel_separation>0.17</wheel_separation>                   # the distance between the two wheels
-                <wheel_radius>0.045</wheel_radius>                          # the radius of the wheels
-                <topic>${prefix}cmd_vel</topic>                             # the topic that will be subscribed to receive velocity commands
-                <tf_topic>${prefix}diff_drive/tf</tf_topic>                 # the topic that will be published in the tf message
-                <odom_topic>${prefix}odom</odom_topic>                      # the topic that will be published in the odometry message
-                <frame_id>${prefix}odom</frame_id>                          # the frame that will be published in the odometry message
-                <child_frame_id>${prefix}base_footprint</child_frame_id>    # the frame that will be published in the odometry message
-                <odom_publish_frequency>50</odom_publish_frequency>         # publish odometry at 50 Hz
-                <max_angular_acceleration>1.2</max_angular_acceleration>    # the maximum angular acceleration of the robot
-                <max_angular_velocity>13.0</max_angular_velocity>           # the maximum angular velocity of the robot
+            <plugin filename="gz-sim-diff-drive-system"
+                    name="ignition::gazebo::systems::DiffDrive">
+                <left_joint>${prefix}wheel_l_joint</left_joint>
+                <right_joint>${prefix}wheel_r_joint</right_joint>
+                <wheel_separation>0.17</wheel_separation>
+                <wheel_radius>0.045</wheel_radius>
+                <topic>${prefix}cmd_vel</topic>
+                <tf_topic>${prefix}diff_drive/tf</tf_topic>
+                <odom_topic>${prefix}odom</odom_topic>
+                <frame_id>${prefix}odom</frame_id>
+                <child_frame_id>${prefix}base_footprint</child_frame_id>
+                <odom_publish_frequency>50</odom_publish_frequency>
+                <max_angular_acceleration>1.2</max_angular_acceleration>
+                <max_angular_velocity>13.0</max_angular_velocity>
             </plugin>
-            <plugin filename="gz-sim-joint-state-publisher-system" name="gz::sim::systems::JointStatePublisher"/>
-                <topic>${prefix}joint_states</topic>                        # the topic that will be published in the joint states message
-                <update_rate>50</update_rate>                               # publish joint states at 50 Hz
-                <joint_name>${prefix}wheel_left_joint</joint_name>          # the joint that will be published in the joint states message
-                <joint_name>${prefix}wheel_right_joint</joint_name>         # the joint that will be published in the joint states message
+            <plugin filename="gz-sim-joint-state-publisher-system"
+                    name="ignition::gazebo::systems::JointStatePublisher">
+                <topic>${prefix}joint_states</topic>
+                <update_rate>50</update_rate>
+                <joint_name>${prefix}wheel_l_joint</joint_name>
+                <joint_name>${prefix}wheel_r_joint</joint_name>
             </plugin>
         </gazebo>

Commit message: Fix-Rviz&Gazebo

File: puzzlebot_description/urdf/puzzlebot.urdf.xacro (robot description, xacro)
@@ -83,21 +83,4 @@
     </collision>
   </link>
-  <link name="laser_link">
-    <inertial>
-      <mass value="0.05"/>
-      <inertia ixx="0.0005" iyy="0.0005" izz="0.0005" ixy="0.0" ixz="0.0" iyz="0.0"/>
-    </inertial>
-    <visual>
-      <geometry>
-        <cylinder radius="0.03" length="0.04"/>
-      </geometry>
-      <material name="black"/>
-    </visual>
-    <collision>
-      <geometry>
-        <cylinder radius="0.03" length="0.04"/>
-      </geometry>
-    </collision>
-  </link>
   <joint name="base_link_joint" type="fixed">
     <parent link="base_footprint"/>
@@ -122,55 +105,4 @@
     <origin xyz="-0.095 0.0 -0.043"/>
   </joint>
-  <joint name="laser_joint" type="fixed">
-    <parent link="base_link"/>
-    <child link="laser_link"/>
-    <origin xyz="0 0 0.1"/>
-  </joint>
-  <gazebo reference="laser_link">
-    <sensor name="laser_sensor" type="gpu_ray">
-      <pose>0 0 0 0 0 0</pose>
-      <ray>
-        <scan>
-          <horizontal>
-            <samples>360</samples>
-            <resolution>1</resolution>
-            <min_angle>-3.14159</min_angle>
-            <max_angle>3.14159</max_angle>
-          </horizontal>
-        </scan>
-        <range>
-          <min>0.12</min>
-          <max>12.0</max>
-          <resolution>0.01</resolution>
-        </range>
-      </ray>
-      <plugin filename="gz-sim-sensors-system" name="gz::sim::systems::Sensors">
-        <render_engine>ogre2</render_engine>
-      </plugin>
-      <always_on>1</always_on>
-      <visualize>true</visualize>
-      <topic>scan</topic>
-      <frame_id>laser_link</frame_id>
-    </sensor>
-  </gazebo>
-  <gazebo>
-    <plugin filename="gz-sim-diff-drive-system" name="gz::sim::systems::DiffDrive">
-      <left_joint>wheel_l_joint</left_joint>
-      <right_joint>wheel_r_joint</right_joint>
-      <wheel_separation>0.19</wheel_separation>
-      <wheel_radius>0.033</wheel_radius>
-      <odom_publish_frequency>50</odom_publish_frequency>
-      <topic>cmd_vel</topic>
-      <odom_topic>odom</odom_topic>
-      <tf_topic>tf</tf_topic>
-      <frame_id>odom</frame_id>
-      <child_frame_id>base_footprint</child_frame_id>
-    </plugin>
-    <plugin filename="gz-sim-joint-state-publisher-system" name="gz::sim::systems::JointStatePublisher">
-      <topic>joint_states</topic>
-      <joint_name>wheel_l_joint</joint_name>
-      <joint_name>wheel_r_joint</joint_name>
-    </plugin>
-  </gazebo>
   <gazebo reference="wheel_l_link">
     <mu1>0.7</mu1>
@@ -191,5 +123,4 @@
     <material>Gazebo/Green</material>
   </gazebo>
-  <xacro:include filename="$(find puzzlebot_description)/urdf/sensor.xacro"/>
   <xacro:puzzlebot_control prefix="$(arg prefix)"/>
   <xacro:rpi_lidar_sensor prefix="$(arg prefix)"/>

Commit message: Really Functional Nav2Goal:)

File: puzzlebot_description/urdf/puzzlebot.urdf.xacro (robot description, xacro)
@@ -15,5 +15,5 @@
     </inertial>
     <visual>
-      <origin xyz="0 0 0" rpy="0 0 0"/>
+      <origin xyz="-0.052 0 0" rpy="0 0 0"/>
       <geometry>
         <mesh filename="file://$(find puzzlebot_description)/meshes/Puzzlebot_Jetson_Lidar_Edition_Base.stl" scale="1 1 1"/>
@@ -22,5 +22,5 @@
     </visual>
     <collision>
-      <origin xyz="0 0 0" rpy="0 0 0"/>
+      <origin xyz="-0.052 0 0" rpy="0 0 0"/>
       <geometry>
         <mesh filename="file://$(find puzzlebot_description)/meshes/Puzzlebot_Jetson_Lidar_Edition_Base.stl" scale="1 1 1"/>
@@ -86,10 +86,10 @@
     <parent link="base_footprint"/>
     <child link="base_link"/>
-    <origin xyz="0 0 0.05"/>
+    <origin xyz="0.052 0 0.05"/>
   </joint>
   <joint name="wheel_r_joint" type="continuous">
     <parent link="base_link"/>
     <child link="wheel_r_link"/>
-    <origin xyz="0.052 -0.095 -0.0025"/>
+    <origin xyz="0.0 -0.095 -0.0025"/>
     <axis xyz="0 1 0"/>
   </joint>
@@ -97,5 +97,5 @@
     <parent link="base_link"/>
     <child link="wheel_l_link"/>
-    <origin xyz="0.052 0.095 -0.0025"/>
+    <origin xyz="0.0 0.095 -0.0025"/>
     <axis xyz="0 1 0"/>
   </joint>
@@ -103,5 +103,5 @@
     <parent link="base_link"/>
     <child link="caster_link"/>
-    <origin xyz="-0.095 0.0 -0.043"/>
+    <origin xyz="-0.147 0.0 -0.043"/>
   </joint>
   <gazebo reference="wheel_l_link">

File: puzzlebot_description/urdf/sensor.xacro (robot description, xacro)
@@ -29,5 +29,5 @@
     lidar_base_mesh_pos_p:='0.0'
     lidar_base_mesh_pos_w:='0.0'
-    lidar_base_pos_x:='0.0425'
+    lidar_base_pos_x:='0.0'
     lidar_base_pos_y:='0.00'
     lidar_base_pos_z:='0.070'

File: puzzlebot_description/urdf/sensor_properties.xacro (robot description, xacro)
@@ -158,5 +158,5 @@
             <xacro:property name="jetson_mesh_pos_w" value="0.0"/>
         <!--jetson Joint parameters-->
-            <xacro:property name="jetson_pos_x" value="0.035"/>
+            <xacro:property name="jetson_pos_x" value="0.0"/>
             <xacro:property name="jetson_pos_y" value="-0.003"/>
             <xacro:property name="jetson_pos_z" value="${chassis_height/2}"/>
